File: ps2usb.kicad_sch (KiCad schematic)
At the start: 12 parts

Commit message: HW 1.2
Parts:
- LED1, R1: footprint Resistor_SMD:R_0805_Medved -> Libs:R_0805_Medved
- PS/2: footprint (none) -> Libs:Connector_Mini-DIN_Female_6Pin_2rows
- RZ1: footprint mcu:rp2040-zero-tht -> Libs:rp2040-zero-tht
Changed lines of the file:
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@@
 			)
 		)
-		(property "Footprint" "mcu:rp2040-zero-tht"
+		(property "Footprint" "Libs:rp2040-zero-tht"
 			(at 130.4641 71.12 0)
 			(effects
@@
 			)
 		)
-		(property "Footprint" "Resistor_SMD:R_0805_Medved"
+		(property "Footprint" "Libs:R_0805_Medved"
 			(at 43.18 80.01 90)
 			(effects
@@
 			)
 		)
-		(property "Footprint" ""
+		(property "Footprint" "Libs:Connector_Mini-DIN_Female_6Pin_2rows"
 			(at 68.58 55.88 0)
 			(effects
@@
 			)
 		)
-		(property "Footprint" "Resistor_SMD:R_0805_Medved"
+		(property "Footprint" "Libs:R_0805_Medved"
 			(at 52.832 80.01 90)
 			(effects
